File: SmartSpeaker/Speaker/Speaker.kicad_sch (KiCad schematic)
At the start: 25 parts, among them J102 Screw_Terminal_01x03, J103 Screw_Terminal_01x02, Q1 DMG2305UX-13, U1 LM384, U2 LTC1655LCN8, U4 LM4040LP-3

Commit message: add potentiometer, prepare to make traces wider
Parts:
- removed JP101: Jumper_2_Bridged, TestPoint:TestPoint_2Pads_Pitch2.54mm_Drill0.8mm, symbol Jumper:Jumper_2_Bridged
- added RV1: R_Potentiometer_Trim, Potentiometer_THT:Potentiometer_Bourns_3296W_Vertical, symbol Device:R_Potentiometer_Trim
Connections:
- net GND: now also RV1.2
- net at U2.7 (VOUT): now also RV1.3
- net at C6.1: now also RV1.1
Changed lines of the file:
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@@
 	(wire
 		(pts
-			(xy 144.78 90.17) (xy 144.78 91.44)
+			(xy 144.78 88.9) (xy 144.78 91.44)
 		)
 		(stroke
@@
 	(wire
 		(pts
-			(xy 144.78 78.74) (xy 144.78 80.01)
-		)
-		(stroke
-			(width 0)
-			(type default)
-		)
-	)
-	(wire
-		(pts
 			(xy 114.3 114.3) (xy 121.92 114.3)
 		)
@@
 		(pts
 			(xy 241.3 80.01) (xy 219.71 80.01)
+		)
+		(stroke
+			(width 0)
+			(type default)
+		)
+	)
+	(wire
+		(pts
+			(xy 144.78 78.74) (xy 144.78 81.28)
 		)
 		(stroke
@@
 				(path "/2bdc2aeb-60f6-455a-ba99-f41f429639a9"
 					(reference "TP102")
+					(unit 1)
+				)
+			)
+		)
+	)
+	(symbol
+		(lib_id "Device:R_Potentiometer_Trim")
+		(at 144.78 85.09 0)
+		(unit 1)
+		(exclude_from_sim no)
+		(in_bom yes)
+		(on_board yes)
+		(dnp no)
+		(fields_autoplaced yes)
+		(property "Reference" "RV1"
+			(at 142.24 83.8199 0)
+			(effects
+				(font
+					(size 1.27 1.27)
+				)
+				(justify right)
+			)
+		)
+		(property "Value" "R_Potentiometer_Trim"
+			(at 142.24 86.3599 0)
+			(effects
+				(font
+					(size 1.27 1.27)
+				)
+				(justify right)
+			)
+		)
+		(property "Footprint" "Potentiometer_THT:Potentiometer_Bourns_3296W_Vertical"
+			(at 144.78 85.09 0)
+			(effects
+				(font
+					(size 1.27 1.27)
+				)
+				(hide yes)
+			)
+		)
+		(property "Datasheet" "~"
+			(at 144.78 85.09 0)
+			(effects
+				(font
+					(size 1.27 1.27)
+				)
+				(hide yes)
+			)
+		)
+		(property "Description" "Trim-potentiometer"
+			(at 144.78 85.09 0)
+			(effects
+				(font
+					(size 1.27 1.27)
+				)
+				(hide yes)
+			)
+		)
+		(pin "3"
+		)
+		(pin "2"
+		)
+		(pin "1"
+		)
+		(instances
+			(project ""
+				(path "/2bdc2aeb-60f6-455a-ba99-f41f429639a9"
+					(reference "RV1")
 					(unit 1)
 				)
@@
 	)
 	(symbol
+		(lib_id "power:GND")
+		(at 148.59 85.09 0)
+		(unit 1)
+		(exclude_from_sim no)
+		(in_bom yes)
+		(on_board yes)
+		(dnp no)
+		(fields_autoplaced yes)
+		(property "Reference" "#PWR0102"
+			(at 148.59 91.44 0)
+			(effects
+				(font
+					(size 1.27 1.27)
+				)
+				(hide yes)
+			)
+		)
+		(property "Value" "GND"
+			(at 148.59 90.17 0)
+			(effects
+				(font
+					(size 1.27 1.27)
+				)
+			)
+		)
+		(property "Footprint" ""
+			(at 148.59 85.09 0)
+			(effects
+				(font
+					(size 1.27 1.27)
+				)
+				(hide yes)
+			)
+		)
+		(property "Datasheet" ""
+			(at 148.59 85.09 0)
+			(effects
+				(font
+					(size 1.27 1.27)
+				)
+				(hide yes)
+			)
+		)
+		(property "Description" "Power symbol creates a global label with name \"GND\" , ground"
+			(at 148.59 85.09 0)
+			(effects
+				(font
+					(size 1.27 1.27)
+				)
+				(hide yes)
+			)
+		)
+		(pin "1"
+		)
+		(instances
+			(project "Speaker"
+				(path "/2bdc2aeb-60f6-455a-ba99-f41f429639a9"
+					(reference "#PWR0102")
+					(unit 1)
+				)
+			)
+		)
+	)
+	(symbol
 		(lib_id "Connector:TestPoint")
 		(at 156.21 78.74 180)
@@
 					(unit 1)
 				)
-			)
-		)
-	)
-	(symbol
-		(lib_id "Jumper:Jumper_2_Bridged")
-		(at 144.78 85.09 90)
-		(unit 1)
-		(exclude_from_sim yes)
-		(in_bom yes)
-		(on_board yes)
-		(dnp no)
-		(fields_autoplaced yes)
-		(property "Reference" "JP101"
-			(at 146.05 83.8199 90)
-			(effects
-				(font
-					(size 1.27 1.27)
-				)
-				(justify right)
-			)
-		)
-		(property "Value" "Jumper_2_Bridged"
-			(at 146.05 86.3599 90)
-			(effects
-				(font
-					(size 1.27 1.27)
-				)
-				(justify right)
-			)
-		)
-		(property "Footprint" "TestPoint:TestPoint_2Pads_Pitch2.54mm_Drill0.8mm"
-			(at 144.78 85.09 0)
-			(effects
-				(font
-					(size 1.27 1.27)
-				)
-				(hide yes)
-			)
-		)
-		(property "Datasheet" "~"
-			(at 144.78 85.09 0)
-			(effects
-				(font
-					(size 1.27 1.27)
-				)
-				(hide yes)
-			)
-		)
-		(property "Description" "Jumper, 2-pole, closed/bridged"
-			(at 144.78 85.09 0)
-			(effects
-				(font
-					(size 1.27 1.27)
-				)
-				(hide yes)
-			)
-		)
-		(pin "1"
-		)
-		(pin "2"
-		)
-		(instances
-			(project ""
-				(path "/2bdc2aeb-60f6-455a-ba99-f41f429639a9"
-					(reference "JP101")
-					(unit 1)
-				)

Commit message: lots of small improvements
Parts:
- added TP8: DAC_Out, TestPoint:TestPoint_THTPad_D2.5mm_Drill1.2mm, symbol Connector:TestPoint
- J1: renamed from J103; value Screw_Terminal_01x02 -> Terminal_2
- J2: renamed from J102; value Screw_Terminal_01x03 -> Terminal_3
- JP1: renamed from JP104; value Jumper_2_Bridged -> Jumper_NC
- JP2: renamed from JP102; value Jumper_2_Bridged -> Jumper_NC
- JP3: renamed from JP103; value Jumper_2_Bridged -> Jumper_NC
- RV1: value R_Potentiometer_Trim -> Trim_Pot
- TP10: renamed from TP7; value TestPoint -> MicIn
- TP5: value TestPoint -> AmpOut
- TP6: value TestPoint -> AmpIn
- TP7: renamed from TP102; value TestPoint -> 3V_Ref
- TP9: renamed from TP101; value TestPoint -> DAC_Ref
- renumbered C7 to C1, C3 to C2, C5 to C3, C6 to C5, C10 to C6, U4 to U2, U2 to U4
Connections:
- net at RV1.3, U4.7 (VOUT): now also TP8.1
Other:
- moved on the sheet: TP9
