File: SmartSpeaker/Speaker/Speaker.kicad_sch (KiCad schematic)
At the start: 26 parts, among them J1 Terminal_2, J2 Terminal_3, Q1 DMG2305UX-13, U1 LM384, U2 LM4040LP-3, U4 LTC1655LCN8

Commit message: lots of improvements, many semi-cosmetic
Parts:
- added H1, H2, H3, H4: MountingHole_Pad, MountingHole:MountingHole_3.2mm_M3_Pad, symbol Mechanical:MountingHole_Pad
Connections:
- net GND: now also H1.1, H2.1, H3.1, H4.1

Commit message: updates per wey
Parts:
- RV1: symbol Device:R_Potentiometer_Trim -> Device:R_Potentiometer_Trim_US
- U2: footprint Package_TO_SOT_THT:TO-92_Inline -> Package_TO_SOT_THT:TO-92_Inline_Wide
Connections:
- net GND: now also A1.32 (GP27), RV1.1; no longer RV1.2
- net at C5.1: now also RV1.2; no longer RV1.1
Changed lines of the file:
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@@
 	(wire
 		(pts
+			(xy 142.24 78.74) (xy 142.24 80.01)
+		)
+		(stroke
+			(width 0)
+			(type default)
+		)
+	)
+	(wire
+		(pts
 			(xy 160.02 76.2) (xy 160.02 78.74)
 		)
@@
 	(wire
 		(pts
-			(xy 104.14 118.11) (xy 101.6 118.11)
+			(xy 105.41 118.11) (xy 101.6 118.11)
 		)
 		(stroke
@@
 	(wire
 		(pts
-			(xy 110.49 124.46) (xy 104.14 124.46)
+			(xy 110.49 124.46) (xy 105.41 124.46)
 		)
 		(stroke
@@
 	(wire
 		(pts
-			(xy 144.78 88.9) (xy 144.78 91.44)
-		)
-		(stroke
-			(width 0)
-			(type default)
-		)
-	)
-	(wire
-		(pts
 			(xy 50.8 130.81) (xy 50.8 133.35)
 		)
@@
 	(wire
 		(pts
+			(xy 104.14 127) (xy 104.14 120.65)
+		)
+		(stroke
+			(width 0)
+			(type default)
+		)
+	)
+	(wire
+		(pts
 			(xy 137.16 92.71) (xy 119.38 92.71)
 		)
@@
 	(wire
 		(pts
+			(xy 144.78 78.74) (xy 144.78 87.63)
+		)
+		(stroke
+			(width 0)
+			(type default)
+		)
+	)
+	(wire
+		(pts
 			(xy 241.3 59.69) (xy 218.44 59.69)
 		)
@@
 	(wire
 		(pts
+			(xy 142.24 78.74) (xy 139.7 78.74)
+		)
+		(stroke
+			(width 0)
+			(type default)
+		)
+	)
+	(wire
+		(pts
 			(xy 190.5 66.04) (xy 193.04 66.04)
 		)
@@
 	(wire
 		(pts
-			(xy 144.78 91.44) (xy 152.4 91.44)
+			(xy 104.14 120.65) (xy 101.6 120.65)
+		)
+		(stroke
+			(width 0)
+			(type default)
+		)
+	)
+	(wire
+		(pts
+			(xy 139.7 91.44) (xy 152.4 91.44)
 		)
 		(stroke
@@
 	(wire
 		(pts
+			(xy 139.7 78.74) (xy 139.7 83.82)
+		)
+		(stroke
+			(width 0)
+			(type default)
+		)
+	)
+	(wire
+		(pts
 			(xy 101.6 82.55) (xy 127 82.55)
 		)
@@
 	(wire
 		(pts
-			(xy 144.78 78.74) (xy 144.78 81.28)
+			(xy 135.89 59.69) (xy 121.92 59.69)
 		)
 		(stroke
@@
 	(wire
 		(pts
-			(xy 135.89 59.69) (xy 121.92 59.69)
+			(xy 101.6 26.67) (xy 156.21 26.67)
 		)
 		(stroke
@@
 	(wire
 		(pts
-			(xy 101.6 26.67) (xy 156.21 26.67)
+			(xy 153.67 64.77) (xy 153.67 71.12)
 		)
 		(stroke
@@
 	(wire
 		(pts
-			(xy 153.67 64.77) (xy 153.67 71.12)
+			(xy 50.8 143.51) (xy 50.8 146.05)
 		)
 		(stroke
@@
 	(wire
 		(pts
-			(xy 50.8 143.51) (xy 50.8 146.05)
+			(xy 173.99 140.97) (xy 125.73 140.97)
 		)
 		(stroke
@@
 	(wire
 		(pts
-			(xy 173.99 140.97) (xy 125.73 140.97)
+			(xy 104.14 40.64) (xy 104.14 44.45)
 		)
 		(stroke
@@
 	(wire
 		(pts
-			(xy 104.14 40.64) (xy 104.14 44.45)
+			(xy 144.78 87.63) (xy 143.51 87.63)
 		)
 		(stroke
@@
 	(wire
 		(pts
-			(xy 104.14 118.11) (xy 104.14 124.46)
+			(xy 105.41 118.11) (xy 105.41 124.46)
 		)
 		(stroke
@@
 	)
 	(symbol
+		(lib_id "power:GND")
+		(at 104.14 127 0)
+		(unit 1)
+		(exclude_from_sim no)
+		(in_bom yes)
+		(on_board yes)
+		(dnp no)
+		(fields_autoplaced yes)
+		(property "Reference" "#PWR014"
+			(at 104.14 133.35 0)
+			(effects
+				(font
+					(size 1.27 1.27)
+				)
+				(hide yes)
+			)
+		)
+		(property "Value" "GND"
+			(at 104.14 132.08 0)
+			(effects
+				(font
+					(size 1.27 1.27)
+				)
+			)
+		)
+		(property "Footprint" ""
+			(at 104.14 127 0)
+			(effects
+				(font
+					(size 1.27 1.27)
+				)
+				(hide yes)
+			)
+		)
+		(property "Datasheet" ""
+			(at 104.14 127 0)
+			(effects
+				(font
+					(size 1.27 1.27)
+				)
+				(hide yes)
+			)
+		)
+		(property "Description" "Power symbol creates a global label with name \"GND\" , ground"
+			(at 104.14 127 0)
+			(effects
+				(font
+					(size 1.27 1.27)
+				)
+				(hide yes)
+			)
+		)
+		(pin "1"
+		)
+		(instances
+			(project "Speaker"
+				(path "/2bdc2aeb-60f6-455a-ba99-f41f429639a9"
+					(reference "#PWR014")
+					(unit 1)
+				)
+			)
+		)
+	)
+	(symbol
 		(lib_id "Amplifier_Audio:LM384")
 		(at 170.18 73.66 0)
@@
 	)
 	(symbol
-		(lib_id "Device:R_Potentiometer_Trim")
-		(at 144.78 85.09 0)
+		(lib_id "Device:R_Potentiometer_Trim_US")
+		(at 139.7 87.63 0)
 		(unit 1)
 		(exclude_from_sim no)
@@
 		(fields_autoplaced yes)
 		(property "Reference" "RV1"
-			(at 142.24 83.8199 0)
+			(at 137.16 86.3599 0)
 			(effects
 				(font
@@
 		)
 		(property "Value" "Trim_Pot"
-			(at 142.24 86.3599 0)
+			(at 137.16 88.8999 0)
 			(effects
 				(font
@@
 		)
 		(property "Footprint" "Potentiometer_THT:Potentiometer_Bourns_3296W_Vertical"
-			(at 144.78 85.09 0)
+			(at 139.7 87.63 0)
 			(effects
 				(font
@@
 		)
 		(property "Datasheet" "~"
-			(at 144.78 85.09 0)
+			(at 139.7 87.63 0)
 			(effects
 				(font
@@
 		)
 		(property "Description" "Trim-potentiometer"
-			(at 144.78 85.09 0)
+			(at 139.7 87.63 0)
 			(effects
 				(font
@@
 		(on_board yes)
 		(dnp no)
-		(fields_autoplaced yes)
 		(property "Reference" "H4"
 			(at 62.23 171.4499 0)
@@
 		)
 		(property "Value" "MountingHole_Pad"
-			(at 62.23 173.9899 0)
+			(at 59.69 168.148 0)
 			(effects
 				(font
@@
 			)
 		)
-		(property "Footprint" "Package_TO_SOT_THT:TO-92_Inline"
+		(property "Footprint" "Package_TO_SOT_THT:TO-92_Inline_Wide"
 			(at 109.22 91.44 0)
 			(effects
@@
 	(symbol
 		(lib_id "power:GND")
-		(at 148.59 85.09 0)
+		(at 142.24 80.01 0)
 		(unit 1)
 		(exclude_from_sim no)
@@
 		(fields_autoplaced yes)
 		(property "Reference" "#PWR06"
-			(at 148.59 91.44 0)
+			(at 142.24 86.36 0)
 			(effects
 				(font
@@
 		)
 		(property "Value" "GND"
-			(at 148.59 90.17 0)
+			(at 142.24 85.09 0)
 			(effects
 				(font
@@
 		)
 		(property "Footprint" ""
-			(at 148.59 85.09 0)
+			(at 142.24 80.01 0)
 			(effects
 				(font
@@
 		)
 		(property "Datasheet" ""
-			(at 148.59 85.09 0)
+			(at 142.24 80.01 0)
 			(effects
 				(font
@@
 		)
 		(property "Description" "Power symbol creates a global label with name \"GND\" , ground"
-			(at 148.59 85.09 0)
+			(at 142.24 80.01 0)
 			(effects
 				(font
@@
 		(on_board yes)
 		(dnp no)
-		(fields_autoplaced yes)
 		(property "Reference" "#PWR07"
 			(at 104.14 101.6 0)

Commit message: Edit PCB to fix issues: - Enlarge OSHW logo - Rotate footprints for screw terminals - Fix pad numbers for barrel jack
Changed lines of the file:
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@@
 (kicad_sch
-	(version 20231120)
+	(version 20250114)
 	(generator "eeschema")
-	(generator_version "8.0")
+	(generator_version "9.0")
 	(paper "A4")
+	(text "DAC's \"output can drive 1000pf without going into oscillation\" applies to cap. to ground; with our cap structure, it doesn't apply"
+		(exclude_from_sim no)
+		(at 218.694 113.538 0)
+		(effects
+			(font
+				(size 1.27 1.27)
+			)
+		)
+	)
+	(text "connect with long-ish jumpers"
+		(exclude_from_sim no)
+		(at 112.268 161.29 0)
+		(effects
+			(font
+				(size 1.27 1.27)
+			)
+		)
+	)
+	(text "VBUS is the usb power input; when it is high, disconnect VSYS to avoid back power"
+		(exclude_from_sim no)
+		(at 120.904 56.134 0)
+		(effects
+			(font
+				(size 1.27 1.27)
+			)
+		)
+	)
 	(junction
 		(at 110.49 140.97)
@@
 		)
 	)
-	(text "DAC's \"output can drive 1000pf without going into oscillation\" applies to cap. to ground; with our cap structure, it doesn't apply"
-		(exclude_from_sim no)
-		(at 218.694 113.538 0)
-		(effects
-			(font
-				(size 1.27 1.27)
-			)
-		)
-	)
-	(text "connect with long-ish jumpers"
-		(exclude_from_sim no)
-		(at 112.268 161.29 0)
-		(effects
-			(font
-				(size 1.27 1.27)
-			)
-		)
-	)
-	(text "VBUS is the usb power input; when it is high, disconnect VSYS to avoid back power"
-		(exclude_from_sim no)
-		(at 120.904 56.134 0)
-		(effects
-			(font
-				(size 1.27 1.27)
-			)
-		)
-	)
 	(label "SpeakerOut"
 		(at 222.25 59.69 0)
@@
 		(at 173.99 137.16)
 		(size 25.4 24.13)
+		(exclude_from_sim no)
+		(in_bom yes)
+		(on_board yes)
+		(dnp no)
 		(stroke
 			(width 0.1524)
@@
 		(at 34.29 15.24)
 		(size 67.31 36.83)
+		(exclude_from_sim no)
+		(in_bom yes)
+		(on_board yes)
+		(dnp no)
 		(fields_autoplaced yes)
 		(stroke
@@
 		)
 	)
+	(embedded_fonts no)
 )
