File: SmartSpeaker/Speaker/Speaker.kicad_pcb (KiCad board)
At the start: 2 copper layers, 94 x 85.1 mm, 47 parts, among them J1 Terminal_2, J2 Terminal_3, J3 54-00166, Q1 DMG2305UX-13, U1 LM384, U2 LM4040LP-3, U3 LM2675N-5, U4 LTC1655LCN8

Commit message: Edit PCB to fix issues: - Enlarge OSHW logo - Rotate footprints for screw terminals - Fix pad numbers for barrel jack
Parts:
- removed the REF** at (134.1, 98.0)
- added REF**: OSHW-Logo2_9.8x8mm_SilkScreen, Symbol:OSHW-Logo2_9.8x8mm_SilkScreen, F.Cu at (133.8, 96.5)
- moved J2 6.95 mm to (67.9, 67.3), turned to -90 degrees
- moved J1 3.57 mm to (121.7, 94.0), turned to 90 degrees
Routing:
- net /Adafruit_1713_Microphone/OUTPUT: track 33.7 -> 27.3 mm
- net /SpeakerOut: track 15.1 -> 18.8 mm
- net VDD: track 61.1 -> 58.2 mm
Other:
- board text added: "SALE System: Smart Speaker Rev B. Calum McConnell"
- board text removed: "SALE System: Smart Speaker Rev A. Calum McConnell"

Commit message: PCB fixes
Parts:
- moved J2 1.59 mm to (67.8, 65.7)
Routing:
- net VDD: track 58.2 -> 56.6 mm
- net /Adafruit_1713_Microphone/OUTPUT: track 27.3 -> 26.6 mm
